Commit message: [master] Angled kinect support

File: src/airdrone_launch/inherited_from_hector/urdf/quadrotor_with_kinect.urdf.xacro (robot description, xacro)
@@ -12,5 +12,5 @@
     <xacro:include filename="$(find hector_sensors_description)/urdf/kinect_camera.urdf.xacro" />
     <xacro:kinect_camera name="camera" parent="base_link">
-      <origin xyz="0.05 0.0 -0.14" rpy="0 1 0"/>
+      <origin xyz="0.05 0.0 -0.14" rpy="0.0 0.1 -0.785"/>
     </xacro:kinect_camera>
 </robot>

Commit message: [master] Door passing features

File: src/airdrone_launch/inherited_from_hector/urdf/quadrotor_with_kinect.urdf.xacro (robot description, xacro)
@@ -12,5 +12,5 @@
     <xacro:include filename="$(find hector_sensors_description)/urdf/kinect_camera.urdf.xacro" />
     <xacro:kinect_camera name="camera" parent="base_link">
-      <origin xyz="0.05 0.0 -0.14" rpy="0.0 0.1 -0.785"/>
+      <origin xyz="0.05 0.0 -0.14" rpy="0.0 0.0 -0.785"/>
     </xacro:kinect_camera>
 </robot>

Commit message: [master] Put Kinect on its place. Passage finder is now able to detect passages only in ranges from 0.6 to 2.8 metres. This is needed for failsafe operation

File: src/airdrone_launch/inherited_from_hector/urdf/quadrotor_with_kinect.urdf.xacro (robot description, xacro)
@@ -12,5 +12,5 @@
     <xacro:include filename="$(find hector_sensors_description)/urdf/kinect_camera.urdf.xacro" />
     <xacro:kinect_camera name="camera" parent="base_link">
-      <origin xyz="0.05 0.0 -0.14" rpy="0.0 0.0 -0.785"/>
+      <origin xyz="0.1 -0.1 -0.0" rpy="0.0 0.0 -0.785"/>
     </xacro:kinect_camera>
 </robot>
