Commit message: runs; spawn issue

File: src/airdrone_gazebo/drone/plugins/urdf/quadrotor_controller.gazebo.xacro (robot description, xacro)
@@ -4,5 +4,5 @@
     <gazebo>
       <plugin name="quadrotor_controller" filename="libgazebo_ros_control.so">
-        <controlPeriod>0.01</controlPeriod>
+        <controlPeriod>0.001</controlPeriod>
         <robotSimType>hector_quadrotor_controller_gazebo/QuadrotorHardwareSim</robotSimType>
       </plugin>

File: src/airdrone_gazebo/drone/sensors/urdf/asus_camera.urdf.xacro (robot description, xacro)
@@ -17,5 +17,5 @@
           <origin xyz="0 0 0" rpy="0 0 0" />
           <geometry>
-            <mesh filename="package://hector_sensors_description/meshes/asus_camera/asus_camera_simple.dae"/>
+            <mesh filename="package://airdrone_gazebo/drone/sensors/meshes/asus_camera/asus_camera_simple.dae"/>
           </geometry>
         </visual>

File: src/airdrone_gazebo/drone/sensors/urdf/hokuyo_utm30lx.urdf.xacro (robot description, xacro)
@@ -17,5 +17,5 @@
           <origin xyz="0 0 0" rpy="0 0 0" />
           <geometry>
-          <mesh filename="package://hector_sensors_description/meshes/hokuyo_utm30lx/hokuyo_utm_30lx$(optenv TEST_SELF_FILTER).dae"/>
+          <mesh filename="package://airdrone_gazebo/drone/sensors/meshes/hokuyo_utm30lx/hokuyo_utm_30lx$(optenv TEST_SELF_FILTER).dae"/>
         </geometry>
         </visual>
@@ -24,5 +24,4 @@
           <geometry>
           <box size="0.058 0.058 0.087" />
-          <!--<mesh filename="package://hector_sensors_description/meshes/hokuyo_utm30lx/hokuyo_utm_30lx.stl"/>-->
         </geometry>
         </collision>

File: src/airdrone_gazebo/drone/sensors/urdf/kinect_camera.urdf.xacro (robot description, xacro)
@@ -13,5 +13,5 @@
           <origin xyz="0 0 0" rpy="0 0 0" />
           <geometry>
-            <mesh filename="package://hector_sensors_description/meshes/kinect_camera/kinect_camera_simple.dae"/>
+            <mesh filename="package://airdrone_gazebo/drone/sensors/meshes/kinect_camera/kinect_camera_simple.dae"/>
           </geometry>
         </visual>
@@ -19,5 +19,5 @@
           <origin xyz="0 0 0" rpy="0 0 0" />
           <geometry>
-            <mesh filename="package://hector_sensors_description/meshes/kinect_camera/kinect_camera_simple.stl"/>
+            <mesh filename="package://airdrone_gazebo/drone/sensors/meshes/kinect_camera/kinect_camera_simple.stl"/>
           </geometry>
         </collision>
@@ -56,5 +56,5 @@
           <update_rate>20</update_rate>
           <camera>
-            <horizontal_fov>${60 * M_PI/180.0}</horizontal_fov>
+            <horizontal_fov>${57.0 * M_PI/180.0}</horizontal_fov>
             <image>
               <format>R8G8B8</format>
@@ -70,4 +70,5 @@
             <alwaysOn>true</alwaysOn>
             <updateRate>20</updateRate>
+            <cameraName>${name}</cameraName>
             <imageTopicName>${name}/rgb/image_raw</imageTopicName>
             <cameraInfoTopicName>${name}/rgb/camera_info</cameraInfoTopicName>
@@ -76,9 +77,10 @@
             <pointCloudTopicName>${name}/depth/points</pointCloudTopicName>
             <frameName>${name}_depth_optical_frame</frameName>
-            <distortion_k1>0.0</distortion_k1>
-            <distortion_k2>0.0</distortion_k2>
-            <distortion_k3>0.0</distortion_k3>
-            <distortion_t1>0.0</distortion_t1>
-            <distortion_t2>0.0</distortion_t2>
+            <pointCloudCutoff>0.5</pointCloudCutoff>
+            <distortionK1>0.00000000</distortionK1>
+            <distortionK2>0.00000000</distortionK2>
+            <distortionK3>0.00000000</distortionK3>
+            <distortionT1>0.00000000</distortionT1>
+            <distortionT2>0.00000000</distortionT2>
           </plugin>
         </sensor>

File: src/airdrone_gazebo/drone/sensors/urdf/sonar_sensor.urdf.xacro (robot description, xacro)
@@ -17,5 +17,5 @@
         <geometry>
           <!--<box size="0.01 0.01 0.01" /> -->
-          <mesh filename="package://hector_sensors_description/meshes/sonar_sensor/max_sonar_ez4.dae"/>
+          <mesh filename="package://airdrone_gazebo/drone/sensors/meshes/sonar_sensor/max_sonar_ez4.dae"/>
         </geometry>
       </visual>
