Commit message: final port of hector quadrotor to airdrone simulator

File: src/airdrone_gazebo/drone/frame/urdf/quadrotor_base.urdf.xacro (robot description, xacro)
@@ -5,5 +5,11 @@
   <!-- Main quadrotor link -->
   <xacro:macro name="quadrotor_base_macro">
-    <link name="base_stabilized">
+    <link name="base_stabilized"/>
+    <joint name="base_stabilized_to_quadrotor_visual" type = "fixed">
+      <parent link = "base_stabilized"/>
+      <child  link = "quadrotor_visual"/>
+      <origin xyz="0 0 0" rpy="0 0 0" />
+    </joint>
+    <link name="quadrotor_visual">
       <inertial>
         <mass value="1.477" />

Commit message: fixed simulator launch files to make odom->base_link transform publish optional

File: src/airdrone_gazebo/drone/frame/urdf/quadrotor_base.urdf.xacro (robot description, xacro)
@@ -5,10 +5,4 @@
   <!-- Main quadrotor link -->
   <xacro:macro name="quadrotor_base_macro">
-    <link name="base_stabilized"/>
-    <joint name="base_stabilized_to_quadrotor_visual" type = "fixed">
-      <parent link = "base_stabilized"/>
-      <child  link = "quadrotor_visual"/>
-      <origin xyz="0 0 0" rpy="0 0 0" />
-    </joint>
     <link name="quadrotor_visual">
       <inertial>
@@ -31,7 +25,8 @@
     </link>
     <link name="base_link"/>
-    <joint name="base_stabilized_to_base" type = "fixed">
-      <parent link = "base_stabilized"/>
-      <child  link = "base_link"/>
+    <joint name="base_link_to_quadrotor_visual" type = "fixed">
+      <parent link = "base_link"/>
+      <child  link = "quadrotor_visual"/>
+      <origin xyz="0 0 0" rpy="0 0 0" />
     </joint>
     <!-- Sonar height sensor -->

Commit message: added rotation estimation to ransac_slam node

File: src/airdrone_gazebo/drone/frame/urdf/quadrotor_base.urdf.xacro (robot description, xacro)
@@ -5,10 +5,4 @@
   <!-- Main quadrotor link -->
   <xacro:macro name="quadrotor_base_macro">
-    <link name="base_stabilized"/>
-    <joint name="base_stabilized_to_quadrotor_visual" type = "fixed">
-      <parent link = "base_stabilized"/>
-      <child  link = "quadrotor_visual"/>
-      <origin xyz="0 0 0" rpy="0 0 0" />
-    </joint>
     <link name="quadrotor_visual">
       <inertial>
@@ -31,10 +25,11 @@
     </link>
     <link name="base_link"/>
-    <joint name="base_stabilized_to_base" type = "fixed">
-      <parent link = "base_stabilized"/>
-      <child  link = "base_link"/>
+    <joint name="base_link_to_quadrotor_visual" type = "fixed">
+      <parent link = "base_link"/>
+      <child  link = "quadrotor_visual"/>
+      <origin xyz="0 0 0" rpy="0 0 0" />
     </joint>
     <!-- Sonar height sensor -->
-    <xacro:sonar_sensor name="sonar" parent="base_link" ros_topic="sonar_height" update_rate="10" min_range="0.01" max_range="30.0" field_of_view="${40*pi/180}" ray_count="3">
+    <xacro:sonar_sensor name="sonar" parent="base_link" ros_topic="sensors/sonar_height" update_rate="10" min_range="0.01" max_range="30.0" field_of_view="${40*pi/180}" ray_count="3">
       <origin xyz="-0.16 0.0 -0.012" rpy="0 ${90*pi/180} 0"/>
     </xacro:sonar_sensor>

File: src/airdrone_gazebo/drone/plugins/urdf/quadrotor_sensors.gazebo.xacro (robot description, xacro)
@@ -6,5 +6,5 @@
       <updateRate>100.0</updateRate>
       <bodyName>base_link</bodyName>
-      <topicName>raw_imu</topicName>
+      <topicName>sensors/apm/raw_imu</topicName>
       <rpyOffsets>0 0 0</rpyOffsets> <!-- deprecated -->
       <gaussianNoise>0</gaussianNoise>  <!-- deprecated -->
