Commit message: start configuring sensor drivers

File: src/airdrone_gazebo/drone/frame/urdf/quadrotor_with_kinect.urdf.xacro (robot description, xacro)
@@ -16,6 +16,6 @@
     <!-- Downward facing camera -->
     <xacro:include filename="$(find airdrone_gazebo)/drone/sensors/urdf/generic_camera.urdf.xacro" />
-    <xacro:generic_camera name="flow_camera" parent="base_link" ros_topic="flow_camera/image" cam_info_topic="flow_camera/camera_info" update_rate="15" res_x="320" res_y="240" image_format="L8" hfov="90">
-      <origin xyz="0.0 0.0 0.0" rpy="0 ${M_PI/2} 0"/>
+    <xacro:generic_camera name="downward_camera" parent="base_link" ros_topic="/sensors/downward_camera/image" cam_info_topic="/sensors/downward_camera/camera_info" update_rate="15" res_x="320" res_y="240" image_format="L8" hfov="75">
+      <origin xyz="0.0 0.0 -0.14" rpy="0 ${M_PI/2} 0"/>
     </xacro:generic_camera>
 </robot>
